Commit message: Removal of wheel odometry information

File: src/articubot_one/description/gazebo_control.xacro (robot description, xacro)
@@ -14,7 +14,7 @@
             <odometry_frame>odom</odometry_frame>
             <robot_base_frame>base_link</robot_base_frame>
-            <publish_odom>true</publish_odom>
-            <publish_odom_tf>true</publish_odom_tf>
-            <publish_wheel_tf>true</publish_wheel_tf>
+            <publish_odom>false</publish_odom>
+            <publish_odom_tf>false</publish_odom_tf>
+            <publish_wheel_tf>false</publish_wheel_tf>
         </plugin>
     </gazebo>

File: src/articubot_one/description/lidar.xacro (robot description, xacro)
@@ -4,7 +4,9 @@
         <parent link="chassis"/>
         <child link="laser_frame"/>
+        <!-- <child link="laser"/> -->
         <origin xyz="0.122 0 0.212" rpy="0 0 0"/>
     </joint>
     <link name="laser_frame">
+    <!-- <link name="laser"> -->
         <visual>
             <geometry>
@@ -30,4 +32,5 @@
     </link>
     <gazebo reference="laser_frame">
+    <!-- <gazebo reference="laser"> -->
         <material>Gazebo/Black</material>
         <sensor name="laser" type="ray">
@@ -54,4 +57,5 @@
                 <output_type>sensor_msgs/LaserScan</output_type>
                 <frame_name>laser_frame</frame_name>
+                <!-- <frame_name>laser</frame_name> -->
             </plugin>
         </sensor>

File: src/articubot_one/description/robot.urdf.xacro (robot description, xacro)
@@ -12,5 +12,3 @@
     <xacro:include filename="lidar.xacro" />
     <xacro:include filename="camera.xacro" />
-    <!-- <xacro:include filename="depth_camera.xacro" /> -->
-    <!-- <xacro:include filename="face.xacro" /> -->
 </robot>

File: src/articubot_one/description/robot_core.xacro (robot description, xacro)
@@ -148,26 +148,26 @@
         <mu2 value="0.001"/>
     </gazebo>
- <!-- *********************** IMU SENSOR SETUP **************************  -->
 <!-- IMU Link -->
 <joint name="imu_joint" type="fixed">
-    <parent link="base_link"/>
-    <child link="imu_link"/>
-    <origin xyz="0 0 0" rpy="0 0 0"/>
+  <parent link="base_link"/>
+  <child link="imu_link"/>
+  <origin xyz="0 0 0" rpy="0 0 0"/>
 </joint>
-  <gazebo reference="imu_link">
+<link name="imu_link">
+</link>
+<gazebo reference="imu_link">
     <gravity>true</gravity>
     <sensor name="imu_sensor" type="imu">
       <always_on>true</always_on>
-      <update_rate>100</update_rate>
+      <update_rate>30</update_rate>
       <visualize>true</visualize>
       <topic>__default_topic__</topic>
-      <plugin filename="libgazebo_ros_imu_sensor.so" name="imu_plugin">
-        <topicName>imu_data</topicName>
-        <bodyName>imu_link</bodyName>
-        <updateRateHZ>10.0</updateRateHZ>
+      <plugin filename="libgazebo_ros_imu_sensor.so" name="imu">
+        <topicName>imu/data</topicName>
+        <updateRateHZ>30.0</updateRateHZ>
         <gaussianNoise>0.0</gaussianNoise>
         <xyzOffset>0 0 0</xyzOffset>
         <rpyOffset>0 0 0</rpyOffset>
-        <frameName>imu_link</frameName>
+        <frameName>imu_frame</frameName>
         <initialOrientationAsReference>false</initialOrientationAsReference>
       </plugin>
@@ -175,97 +175,19 @@
     </sensor>
   </gazebo>
-<link name="imu_link">
-  <inertial>
-    <mass value="0.01"/>
-    <origin rpy="0 0 0" xyz="0 0 0"/>
-    <inertia ixx="0.001" ixy="0" ixz="0" iyy="0.001" iyz="0" izz="0.001"/>
-  </inertial>
-  <sensor name="bmb_imu" type="imu">
-    <imu>
-      <orientation>
-        <x>
-          <noise type="gaussian" mean="0.0" stddev="2e-3"/>
-        </x>
-        <y>
-          <noise type="gaussian" mean="0.0" stddev="2e-3"/>
-        </y>
-        <z>
-          <noise type="gaussian" mean="0.0" stddev="2e-3"/>
-        </z>
-      </orientation>
-      <angular_velocity>
-        <x>
-          <noise type="gaussian" mean="0.0" stddev="2e-4"/>
-        </x>
-        <y>
-          <noise type="gaussian" mean="0.0" stddev="2e-4"/>
-        </y>
-        <z>
-          <noise type="gaussian" mean="0.0" stddev="2e-4"/>
-        </z>
-      </angular_velocity>
-      <linear_acceleration>
-        <x>
-          <noise type="gaussian" mean="0.0" stddev="1.7e-2"/>
-        </x>
-        <y>
-          <noise type="gaussian" mean="0.0" stddev="1.7e-2"/>
-        </y>
-        <z>
-          <noise type="gaussian" mean="0.0" stddev="1.7e-2"/>
-        </z>
-      </linear_acceleration>
-    </imu>
-    <plugin name="articubot_imu" filename="libgazebo_ros_imu_sensor.so">
-      <ros>
-        <namespace>/imu</namespace>
-        <remapping>~/out:=data</remapping>
-      </ros>
-    </plugin>
-  </sensor>
-</link>
 <!-- GPS Link -->
- <joint name="gps_joint" type="fixed">
+<joint name="gps_joint" type="fixed">
     <parent link="base_link"/>
     <child link="gps_link"/>
     <origin xyz="0 0 0" rpy="0 0 0"/>
 </joint>
+<link name="gps_link">
+</link>
 <gazebo reference="gps_link">
     <sensor name="gps_sensor" type="gps">
         <always_on>true</always_on>
-        <update_rate>1.0</update_rate>
-        <plugin name="gps_controller" filename="libgazebo_ros_gps_sensor.so">
-            <ros>
-                <!-- <namespace>/br</namespace> -->
-                <remapping>gps_controller/out:=gps</remapping>
-            </ros>
-            <frame_name>gps_link</frame_name>
+        <update_rate>10.0</update_rate>
+        <plugin filename="libgazebo_ros_gps_sensor.so" name="gps">
         </plugin>
     </sensor>
-    <material>Gazebo/Grey</material>
 </gazebo>
-<link name="gps_link">
-  <inertial>
-    <mass value="0.01"/>
-    <origin rpy="0 0 0" xyz="0 0 0"/>
-    <inertia ixx="0.001" ixy="0" ixz="0" iyy="0.001" iyz="0" izz="0.001"/>
-  </inertial>
-  <sensor name="bmb_gps" type="gps">
-    <gps>
-      <position_sensing>
-        <horizontal>
-          <noise type="gaussian" mean="0.0" stddev="1e-2"/>
-        </horizontal>
-        <vertical>
-          <noise type="gaussian" mean="0.0" stddev="1"/>
-        </vertical>
-      </position_sensing>
-    </gps>
-    <plugin name="articubot_gps" filename="libgazebo_ros_gps_sensor.so">
-      <ros>
-        <remapping>~/out:=gps/fix</remapping>
-      </ros>
-    </plugin>
-  </sensor>
-</link>
 </robot>
